File: Circuit/Power.sch (KiCad schematic (older format))
At the start: 15 parts, among them Q201 FDN340P, Q202 FDN340P, Q203 FDN340P, U201 CN3063, U202 MCP6002

Commit message: Traces in.
Parts:
- C203: value 100uF 16V X5R -> 220uF 16V
- LED201: value LED_GREEN -> LED_DONE
- LED202: value LED_RED -> LED_CHRG
- R202, R203: value 1K -> 330R
Changed lines of the file:
@@
 SOLAR_IN
 $Comp
-L GND #PWR202
+L GND #PWR032
 U 1 1 563C4E24
 P 4000 4650
-F 0 "#PWR202" H 4000 4400 50  0001 C CNN
+F 0 "#PWR032" H 4000 4400 50  0001 C CNN
 F 1 "GND" H 4000 4500 50  0000 C CNN
 F 2 "" H 4000 4650 60  0000 C CNN
@@
 $EndComp
 $Comp
-L GND #PWR201
+L GND #PWR033
 U 1 1 563C5B2C
 P 1150 1500
-F 0 "#PWR201" H 1150 1250 50  0001 C CNN
+F 0 "#PWR033" H 1150 1250 50  0001 C CNN
 F 1 "GND" H 1150 1350 50  0000 C CNN
 F 2 "" H 1150 1500 60  0000 C CNN
@@
 P 2950 3400
 F 0 "LED202" H 2950 3500 50  0000 C CNN
-F 1 "LED_RED" H 2950 3300 50  0000 C CNN
+F 1 "LED_CHRG" H 2950 3300 50  0000 C CNN
 F 2 "FT:LED-0805" H 2950 3550 24  0000 C CNN
 F 3 "" H 2950 3400 60  0000 C CNN
@@
 P 2950 2800
 F 0 "R203" V 2850 2800 50  0000 C CNN
-F 1 "1K" V 2950 2800 50  0000 C CNN
+F 1 "330R" V 2950 2800 50  0000 C CNN
 F 2 "FT:0805" V 3050 2800 24  0000 C CNN
 F 3 "" H 2950 2800 60  0000 C CNN
@@
 P 2450 3400
 F 0 "LED201" H 2450 3500 50  0000 C CNN
-F 1 "LED_GREEN" H 2450 3300 50  0000 C CNN
+F 1 "LED_DONE" H 2450 3300 50  0000 C CNN
 F 2 "FT:LED-0805" H 2450 3550 24  0000 C CNN
 F 3 "" H 2450 3400 60  0000 C CNN
@@
 P 2450 2800
 F 0 "R202" V 2350 2800 50  0000 C CNN
-F 1 "1K" V 2450 2800 50  0000 C CNN
+F 1 "330R" V 2450 2800 50  0000 C CNN
 F 2 "FT:0805" V 2550 2800 24  0000 C CNN
 F 3 "" H 2450 2800 60  0000 C CNN
@@
 Charging current\nIr = 220mA max
 $Comp
-L GND #PWR204
+L GND #PWR034
 U 1 1 56417FB3
 P 7450 4100
-F 0 "#PWR204" H 7450 3850 50  0001 C CNN
+F 0 "#PWR034" H 7450 3850 50  0001 C CNN
 F 1 "GND" H 7450 3950 50  0000 C CNN
 F 2 "" H 7450 4100 60  0000 C CNN
@@
 VOUT
 $Comp
-L GND #PWR207
+L GND #PWR035
 U 1 1 5641AA9F
 P 10250 2500
-F 0 "#PWR207" H 10250 2250 50  0001 C CNN
+F 0 "#PWR035" H 10250 2250 50  0001 C CNN
 F 1 "GND" H 10250 2350 50  0000 C CNN
 F 2 "" H 10250 2500 60  0000 C CNN
@@
 VOUT
 $Comp
-L GND #PWR205
+L GND #PWR036
 U 1 1 5642C1C1
 P 9000 4100
-F 0 "#PWR205" H 9000 3850 50  0001 C CNN
+F 0 "#PWR036" H 9000 3850 50  0001 C CNN
 F 1 "GND" H 9000 3950 50  0000 C CNN
 F 2 "" H 9000 4100 60  0000 C CNN
@@
 P 10250 2150
 F 0 "C203" H 10275 2250 50  0000 L CNN
-F 1 "100uF 16V X5R" H 10275 2050 50  0000 L CNN
+F 1 "220uF 16V" H 10275 2050 50  0000 L CNN
 F 2 "FT:1210_CAP" H 10400 2350 24  0000 C CNN
 F 3 "" H 10250 2150 60  0000 C CNN
@@
 $EndComp
 $Comp
-L PWR_FLAG #FLG202
+L PWR_FLAG #FLG037
 U 1 1 5642D1CE
 P 10450 1800
-F 0 "#FLG202" H 10450 1895 50  0001 C CNN
+F 0 "#FLG037" H 10450 1895 50  0001 C CNN
 F 1 "PWR_FLAG" H 10450 1980 50  0000 C CNN
 F 2 "" H 10450 1800 60  0000 C CNN
@@
 $EndComp
 $Comp
-L PWR_FLAG #FLG201
+L PWR_FLAG #FLG038
 U 1 1 5642D5A3
 P 3900 1800
-F 0 "#FLG201" H 3900 1895 50  0001 C CNN
+F 0 "#FLG038" H 3900 1895 50  0001 C CNN
 F 1 "PWR_FLAG" H 3900 1980 50  0000 C CNN
 F 2 "" H 3900 1800 60  0000 C CNN
@@
 $EndComp
 $Comp
-L GND #PWR206
+L GND #PWR039
 U 1 1 5642DA26
 P 10000 4150
-F 0 "#PWR206" H 10000 3900 50  0001 C CNN
+F 0 "#PWR039" H 10000 3900 50  0001 C CNN
 F 1 "GND" H 10000 4000 50  0000 C CNN
 F 2 "" H 10000 4150 60  0000 C CNN
@@
 $EndComp
 $Comp
-L GND #PWR203
+L GND #PWR040
 U 1 1 5642CE9D
 P 4600 2350
-F 0 "#PWR203" H 4600 2100 50  0001 C CNN
+F 0 "#PWR040" H 4600 2100 50  0001 C CNN
 F 1 "GND" H 4600 2200 50  0000 C CNN
 F 2 "" H 4600 2350 60  0000 C CNN
@@
 Battery goes here\nin circuit\n(actually connected\nto VBAT on parent sheet)
 Wire Wire Line
-	2950 3600 2950 3650
+	2950 3650 2950 3600
 $EndSCHEMATC
