File: Circuit/ESPlant-Sensors.sch (KiCad schematic (older format))
At the start: 6 parts, among them U401 BME280, U402 ADXL345

Commit message: Downgrade STM32 to cute little TSSOP20 STM32F042F6
Parts:
- renumbered C401 to C301, C402 to C302, R401 to R301, R402 to R302, U401 to U301, U402 to U302
Changed lines of the file:
@@
 EESchema Schematic File Version 2
+LIBS:ESPlant-rescue
 LIBS:freetronics_schematic
 LIBS:power
@@
 $Descr A4 11693 8268
 encoding utf-8
-Sheet 4 4
+Sheet 4 3
 Title ""
 Date ""
@@
 $EndDescr
 $Comp
-L BME280 U401
+L BME280 U301
 U 1 1 564CD8ED
 P 3150 3300
-F 0 "U401" H 3400 3000 60  0000 C CNN
+F 0 "U301" H 3400 3000 60  0000 C CNN
 F 1 "BME280" H 3150 3300 60  0000 C CNN
 F 2 "" H 3150 3300 60  0000 C CNN
@@
 	2450 3150 2450 3250
 $Comp
-L GND #PWR036
+L GND #PWR038
 U 1 1 564CDB3E
 P 2450 3250
-F 0 "#PWR036" H 2450 3000 50  0001 C CNN
+F 0 "#PWR038" H 2450 3000 50  0001 C CNN
 F 1 "GND" H 2450 3100 50  0000 C CNN
 F 2 "" H 2450 3250 60  0000 C CNN
@@
 Connection ~ 2450 2500
 $Comp
-L R R402
+L R R302
 U 1 1 564CDB75
 P 2250 3050
-F 0 "R402" V 2330 3050 50  0000 C CNN
+F 0 "R302" V 2330 3050 50  0000 C CNN
 F 1 "4.7K" V 2250 3050 50  0000 C CNN
 F 2 "" H 2250 3050 60  0000 C CNN
@@
 $EndComp
 $Comp
-L R R401
+L R R301
 U 1 1 564CDBA3
 P 2050 2950
-F 0 "R401" V 2130 2950 50  0000 C CNN
+F 0 "R301" V 2130 2950 50  0000 C CNN
 F 1 "4.7K" V 2050 2950 50  0000 C CNN
 F 2 "" H 2050 2950 60  0000 C CNN
@@
 Connection ~ 3250 2500
 $Comp
-L +3.3V #PWR037
+L +3.3V #PWR039
 U 1 1 564CDC53
 P 3250 2350
-F 0 "#PWR037" H 3250 2200 50  0001 C CNN
+F 0 "#PWR039" H 3250 2200 50  0001 C CNN
 F 1 "+3.3V" H 3250 2490 50  0000 C CNN
 F 2 "" H 3250 2350 60  0000 C CNN
@@
 $EndComp
 $Comp
-L GND #PWR038
+L GND #PWR040
 U 1 1 564CDC6D
 P 3250 4000
-F 0 "#PWR038" H 3250 3750 50  0001 C CNN
+F 0 "#PWR040" H 3250 3750 50  0001 C CNN
 F 1 "GND" H 3250 3850 50  0000 C CNN
 F 2 "" H 3250 4000 60  0000 C CNN
@@
 BME280 Temp/Humidity/Pressure\n
 $Comp
-L ADXL345 U402
+L ADXL345 U302
 U 1 1 564CE29B
 P 6150 3100
-F 0 "U402" H 5600 2550 60  0000 C CNN
+F 0 "U302" H 5600 2550 60  0000 C CNN
 F 1 "ADXL345" H 6150 2850 60  0000 C CNN
 F 2 "" H 6100 2800 60  0000 C CNN
@@
 Connection ~ 5950 2300
 $Comp
-L +3.3V #PWR039
+L +3.3V #PWR041
 U 1 1 564CE661
 P 6150 2200
-F 0 "#PWR039" H 6150 2050 50  0001 C CNN
+F 0 "#PWR041" H 6150 2050 50  0001 C CNN
 F 1 "+3.3V" H 6150 2340 50  0000 C CNN
 F 2 "" H 6150 2200 60  0000 C CNN
@@
 Connection ~ 6150 2300
 $Comp
-L GND #PWR040
+L GND #PWR042
 U 1 1 564CE6B9
 P 6150 4100
-F 0 "#PWR040" H 6150 3850 50  0001 C CNN
+F 0 "#PWR042" H 6150 3850 50  0001 C CNN
 F 1 "GND" H 6150 3950 50  0000 C CNN
 F 2 "" H 6150 4100 60  0000 C CNN
@@
 NoConn ~ 7100 2950
 $Comp
-L C C402
+L C C302
 U 1 1 564CEBB9
 P 4750 2650
-F 0 "C402" H 4775 2750 50  0000 L CNN
+F 0 "C302" H 4775 2750 50  0000 L CNN
 F 1 "1uF 6.3V" H 4400 2550 50  0000 L CNN
 F 2 "" H 4788 2500 30  0000 C CNN
@@
 	4750 2800 4750 2950
 $Comp
-L GND #PWR041
+L GND #PWR043
 U 1 1 564CEC16
 P 4750 2950
-F 0 "#PWR041" H 4750 2700 50  0001 C CNN
+F 0 "#PWR043" H 4750 2700 50  0001 C CNN
 F 1 "GND" H 4750 2800 50  0000 C CNN
 F 2 "" H 4750 2950 60  0000 C CNN
@@
 Connection ~ 5100 2300
 $Comp
-L C C401
+L C C301
 U 1 1 564CEC68
 P 3800 2700
-F 0 "C401" H 3825 2800 50  0000 L CNN
+F 0 "C301" H 3825 2800 50  0000 L CNN
 F 1 "1uF 6.3V" H 3825 2600 50  0000 L CNN
 F 2 "" H 3838 2550 30  0000 C CNN
@@
 	3800 2850 3800 2950
 $Comp
-L GND #PWR042
+L GND #PWR044
 U 1 1 564CED66
 P 3800 2950
-F 0 "#PWR042" H 3800 2700 50  0001 C CNN
+F 0 "#PWR044" H 3800 2700 50  0001 C CNN
 F 1 "GND" H 3800 2800 50  0000 C CNN
 F 2 "" H 3800 2950 60  0000 C CNN

Commit message: Footprint assignment for schematic, including footprints for new parts
Removed on-PCB UV sensor in favour of offboard one.
Parts:
- C301, C302, R301, R302: footprint (none) -> FT:0805
- U301: footprint (none) -> Plant:BME280
- U302: footprint (none) -> Plant:ADXL345
Changed lines of the file:
@@
 F 0 "U301" H 3400 3000 60  0000 C CNN
 F 1 "BME280" H 3150 3300 60  0000 C CNN
-F 2 "" H 3150 3300 60  0000 C CNN
+F 2 "Plant:BME280" H 3150 3200 24  0000 C CNN
 F 3 "" H 3150 3300 60  0000 C CNN
 	1    3150 3300
@@
 	2450 3150 2450 3250
 $Comp
-L GND #PWR038
+L GND #PWR045
 U 1 1 564CDB3E
 P 2450 3250
-F 0 "#PWR038" H 2450 3000 50  0001 C CNN
+F 0 "#PWR045" H 2450 3000 50  0001 C CNN
 F 1 "GND" H 2450 3100 50  0000 C CNN
 F 2 "" H 2450 3250 60  0000 C CNN
@@
 F 0 "R302" V 2330 3050 50  0000 C CNN
 F 1 "4.7K" V 2250 3050 50  0000 C CNN
-F 2 "" H 2250 3050 60  0000 C CNN
+F 2 "FT:0805" V 2350 2850 24  0000 C CNN
 F 3 "" H 2250 3050 60  0000 C CNN
 	1    2250 3050
@@
 F 0 "R301" V 2130 2950 50  0000 C CNN
 F 1 "4.7K" V 2050 2950 50  0000 C CNN
-F 2 "" H 2050 2950 60  0000 C CNN
+F 2 "FT:0805" V 2150 2750 24  0000 C CNN
 F 3 "" H 2050 2950 60  0000 C CNN
 	1    2050 2950
@@
 Connection ~ 3250 2500
 $Comp
-L +3.3V #PWR039
+L +3.3V #PWR046
 U 1 1 564CDC53
 P 3250 2350
-F 0 "#PWR039" H 3250 2200 50  0001 C CNN
+F 0 "#PWR046" H 3250 2200 50  0001 C CNN
 F 1 "+3.3V" H 3250 2490 50  0000 C CNN
 F 2 "" H 3250 2350 60  0000 C CNN
@@
 $EndComp
 $Comp
-L GND #PWR040
+L GND #PWR047
 U 1 1 564CDC6D
 P 3250 4000
-F 0 "#PWR040" H 3250 3750 50  0001 C CNN
+F 0 "#PWR047" H 3250 3750 50  0001 C CNN
 F 1 "GND" H 3250 3850 50  0000 C CNN
 F 2 "" H 3250 4000 60  0000 C CNN
@@
 F 0 "U302" H 5600 2550 60  0000 C CNN
 F 1 "ADXL345" H 6150 2850 60  0000 C CNN
-F 2 "" H 6100 2800 60  0000 C CNN
+F 2 "Plant:ADXL345" H 6100 2800 24  0000 C CNN
 F 3 "" H 6100 2800 60  0000 C CNN
 	1    6150 3100
@@
 Connection ~ 5950 2300
 $Comp
-L +3.3V #PWR041
+L +3.3V #PWR048
 U 1 1 564CE661
 P 6150 2200
-F 0 "#PWR041" H 6150 2050 50  0001 C CNN
+F 0 "#PWR048" H 6150 2050 50  0001 C CNN
 F 1 "+3.3V" H 6150 2340 50  0000 C CNN
 F 2 "" H 6150 2200 60  0000 C CNN
@@
 Connection ~ 6150 2300
 $Comp
-L GND #PWR042
+L GND #PWR049
 U 1 1 564CE6B9
 P 6150 4100
-F 0 "#PWR042" H 6150 3850 50  0001 C CNN
+F 0 "#PWR049" H 6150 3850 50  0001 C CNN
 F 1 "GND" H 6150 3950 50  0000 C CNN
 F 2 "" H 6150 4100 60  0000 C CNN
@@
 F 0 "C302" H 4775 2750 50  0000 L CNN
 F 1 "1uF 6.3V" H 4400 2550 50  0000 L CNN
-F 2 "" H 4788 2500 30  0000 C CNN
+F 2 "FT:0805" H 4500 2500 24  0000 C CNN
 F 3 "" H 4750 2650 60  0000 C CNN
 	1    4750 2650
@@
 	4750 2800 4750 2950
 $Comp
-L GND #PWR043
+L GND #PWR050
 U 1 1 564CEC16
 P 4750 2950
-F 0 "#PWR043" H 4750 2700 50  0001 C CNN
+F 0 "#PWR050" H 4750 2700 50  0001 C CNN
 F 1 "GND" H 4750 2800 50  0000 C CNN
 F 2 "" H 4750 2950 60  0000 C CNN
@@
 F 0 "C301" H 3825 2800 50  0000 L CNN
 F 1 "1uF 6.3V" H 3825 2600 50  0000 L CNN
-F 2 "" H 3838 2550 30  0000 C CNN
+F 2 "FT:0805" H 3900 2550 24  0000 C CNN
 F 3 "" H 3800 2700 60  0000 C CNN
 	1    3800 2700
@@
 	3800 2850 3800 2950
 $Comp
-L GND #PWR044
+L GND #PWR051
 U 1 1 564CED66
 P 3800 2950
-F 0 "#PWR044" H 3800 2700 50  0001 C CNN
+F 0 "#PWR051" H 3800 2700 50  0001 C CNN
 F 1 "GND" H 3800 2800 50  0000 C CNN
 F 2 "" H 3800 2950 60  0000 C CNN

Commit message: Revise schematic for V1.1 based on V1.0 evaluation:
* Swap SDA, SCL on ESP (5,4 to 4,5) to match Arduino default
* Q101 source, drain were swapped
* BME280 change i2c address config  0x76 -> 0x77 (match Adafruit library)
* ADXL345 change i2c address from 0x1d -> 0x53 (match Adafruit library)
* Specify colours for "charging", "done" LEDs in component values
* R202, R203 LED series resistors changed to 1K
* Add GPIO2 pullup to strapping resistors, required for reliable reset
* Add autoreset: connect ESP_RESET to PA7 on STM32, GPIO0 to PB8. Remove
  "ADC5" pin from design.
* Add 1K series resistor between GPIO16 and RESET (replacing solder
  jumper). Otherwise pulling reset line draws >50mA!!
* Add 1K series resistor from GPIO0 to GPIO0 reset button & STM32
  GPIO. This is because GPIO0 defaults to clock output on reset,
  driving a square wave.
* Change 220uF 1210 bulk capacitor value to 100uF, reflecting part
  availability and reliability shown in testing.
Connections:
- net +3V3: now also U301.5 (SDO); no longer U302.12 (SDO/ALT_ADDR)
- net GND: now also U302.12 (SDO/ALT_ADDR); no longer U301.5 (SDO)
Other:
- note added: "I2C Address 0x77\n"
- note removed: "I2C Address 0x76"
Changed lines of the file:
@@
 I2C_SCL
 Wire Wire Line
-	2550 3150 2450 3150
-Wire Wire Line
-	2450 3150 2450 3250
-$Comp
-L GND #PWR301
-U 1 1 564CDB3E
-P 2450 3250
-F 0 "#PWR301" H 2450 3000 50  0001 C CNN
-F 1 "GND" H 2450 3100 50  0000 C CNN
-F 2 "" H 2450 3250 60  0000 C CNN
-F 3 "" H 2450 3250 60  0000 C CNN
-	1    2450 3250
-	1    0    0    -1
-$EndComp
+	2400 3150 2550 3150
 Wire Wire Line
 	3250 2350 3250 2750
@@
 Connection ~ 3250 2500
 $Comp
-L +3.3V #PWR302
+L +3.3V #PWR301
 U 1 1 564CDC53
 P 3250 2350
-F 0 "#PWR302" H 3250 2200 50  0001 C CNN
+F 0 "#PWR301" H 3250 2200 50  0001 C CNN
 F 1 "+3.3V" H 3250 2490 50  0000 C CNN
 F 2 "" H 3250 2350 60  0000 C CNN
@@
 $EndComp
 $Comp
-L GND #PWR303
+L GND #PWR302
 U 1 1 564CDC6D
 P 3250 4000
-F 0 "#PWR303" H 3250 3750 50  0001 C CNN
+F 0 "#PWR302" H 3250 3750 50  0001 C CNN
 F 1 "GND" H 3250 3850 50  0000 C CNN
 F 2 "" H 3250 4000 60  0000 C CNN
@@
 Connection ~ 3250 3950
 Text Notes 1950 3900 0    60   ~ 0
-I2C Address 0x76
+I2C Address 0x77\n
 Text Notes 1800 1750 0    79   ~ 0
 BME280 Temp/Humidity/Pressure\n
@@
 Connection ~ 5950 2300
 $Comp
-L +3.3V #PWR306
+L +3.3V #PWR305
 U 1 1 564CE661
 P 6150 2200
-F 0 "#PWR306" H 6150 2050 50  0001 C CNN
+F 0 "#PWR305" H 6150 2050 50  0001 C CNN
 F 1 "+3.3V" H 6150 2340 50  0000 C CNN
 F 2 "" H 6150 2200 60  0000 C CNN
@@
 Connection ~ 6150 2300
 $Comp
-L GND #PWR307
+L GND #PWR306
 U 1 1 564CE6B9
 P 6150 4100
-F 0 "#PWR307" H 6150 3850 50  0001 C CNN
+F 0 "#PWR306" H 6150 3850 50  0001 C CNN
 F 1 "GND" H 6150 3950 50  0000 C CNN
 F 2 "" H 6150 4100 60  0000 C CNN
@@
 	4750 2800 4750 2950
 $Comp
-L GND #PWR305
+L GND #PWR304
 U 1 1 564CEC16
 P 4750 2950
-F 0 "#PWR305" H 4750 2700 50  0001 C CNN
+F 0 "#PWR304" H 4750 2700 50  0001 C CNN
 F 1 "GND" H 4750 2800 50  0000 C CNN
 F 2 "" H 4750 2950 60  0000 C CNN
@@
 	3800 2850 3800 2950
 $Comp
-L GND #PWR304
+L GND #PWR303
 U 1 1 564CED66
 P 3800 2950
-F 0 "#PWR304" H 3800 2700 50  0001 C CNN
+F 0 "#PWR303" H 3800 2700 50  0001 C CNN
 F 1 "GND" H 3800 2800 50  0000 C CNN
 F 2 "" H 3800 2950 60  0000 C CNN
@@
 Wire Wire Line
 	5300 3150 5000 3150
-Wire Wire Line
-	5000 3150 5000 2300
-Connection ~ 5000 2300
 Text Notes 4700 3900 0    60   ~ 0
 I2C Address 0x53\n
@@
 Text HLabel 7100 2850 2    60   Input ~ 0
 ADXL_INT
+Wire Wire Line
+	2400 3150 2400 2500
+Connection ~ 2400 2500
+Wire Wire Line
+	5000 3150 5000 2900
+Wire Wire Line
+	5000 2900 4750 2900
+Connection ~ 4750 2900
 $EndSCHEMATC

Commit message: Downsize 0805s to 0603 for @jonoxer's pnp machine :)
Parts:
- C301, C302: footprint FT:0805 -> FT:0603_CAP
- R301, R302: footprint FT:0805 -> FT:0603
Changed lines of the file:
@@
 F 0 "R302" V 2330 3050 50  0000 C CNN
 F 1 "4.7K" V 2250 3050 50  0000 C CNN
-F 2 "FT:0805" V 2350 2850 24  0000 C CNN
+F 2 "FT:0603" V 2350 2850 24  0000 C CNN
 F 3 "" H 2250 3050 60  0000 C CNN
 	1    2250 3050
@@
 F 0 "R301" V 2130 2950 50  0000 C CNN
 F 1 "4.7K" V 2050 2950 50  0000 C CNN
-F 2 "FT:0805" V 2150 2750 24  0000 C CNN
+F 2 "FT:0603" V 2150 2750 24  0000 C CNN
 F 3 "" H 2050 2950 60  0000 C CNN
 	1    2050 2950
@@
 Connection ~ 3250 2500
 $Comp
-L +3.3V #PWR301
+L +3.3V #PWR042
 U 1 1 564CDC53
 P 3250 2350
-F 0 "#PWR301" H 3250 2200 50  0001 C CNN
+F 0 "#PWR042" H 3250 2200 50  0001 C CNN
 F 1 "+3.3V" H 3250 2490 50  0000 C CNN
 F 2 "" H 3250 2350 60  0000 C CNN
@@
 $EndComp
 $Comp
-L GND #PWR302
+L GND #PWR043
 U 1 1 564CDC6D
 P 3250 4000
-F 0 "#PWR302" H 3250 3750 50  0001 C CNN
+F 0 "#PWR043" H 3250 3750 50  0001 C CNN
 F 1 "GND" H 3250 3850 50  0000 C CNN
 F 2 "" H 3250 4000 60  0000 C CNN
@@
 Connection ~ 5950 2300
 $Comp
-L +3.3V #PWR305
+L +3.3V #PWR044
 U 1 1 564CE661
 P 6150 2200
-F 0 "#PWR305" H 6150 2050 50  0001 C CNN
+F 0 "#PWR044" H 6150 2050 50  0001 C CNN
 F 1 "+3.3V" H 6150 2340 50  0000 C CNN
 F 2 "" H 6150 2200 60  0000 C CNN
@@
 Connection ~ 6150 2300
 $Comp
-L GND #PWR306
+L GND #PWR045
 U 1 1 564CE6B9
 P 6150 4100
-F 0 "#PWR306" H 6150 3850 50  0001 C CNN
+F 0 "#PWR045" H 6150 3850 50  0001 C CNN
 F 1 "GND" H 6150 3950 50  0000 C CNN
 F 2 "" H 6150 4100 60  0000 C CNN
@@
 F 0 "C302" H 4775 2750 50  0000 L CNN
 F 1 "1uF 6.3V" H 4400 2550 50  0000 L CNN
-F 2 "FT:0805" H 4500 2500 24  0000 C CNN
+F 2 "FT:0603_CAP" H 4500 2500 24  0000 C CNN
 F 3 "" H 4750 2650 60  0000 C CNN
 	1    4750 2650
@@
 	4750 2800 4750 2950
 $Comp
-L GND #PWR304
+L GND #PWR046
 U 1 1 564CEC16
 P 4750 2950
-F 0 "#PWR304" H 4750 2700 50  0001 C CNN
+F 0 "#PWR046" H 4750 2700 50  0001 C CNN
 F 1 "GND" H 4750 2800 50  0000 C CNN
 F 2 "" H 4750 2950 60  0000 C CNN
@@
 F 0 "C301" H 3825 2800 50  0000 L CNN
 F 1 "1uF 6.3V" H 3825 2600 50  0000 L CNN
-F 2 "FT:0805" H 3900 2550 24  0000 C CNN
+F 2 "FT:0603_CAP" H 3900 2550 24  0000 C CNN
 F 3 "" H 3800 2700 60  0000 C CNN
 	1    3800 2700
@@
 	3800 2850 3800 2950
 $Comp
-L GND #PWR303
+L GND #PWR047
 U 1 1 564CED66
 P 3800 2950
-F 0 "#PWR303" H 3800 2700 50  0001 C CNN
+F 0 "#PWR047" H 3800 2700 50  0001 C CNN
 F 1 "GND" H 3800 2800 50  0000 C CNN
 F 2 "" H 3800 2950 60  0000 C CNN
