File: Circuit/ESPlant.kicad_pcb (KiCad board)
At the start: 2 copper layers, 97 x 77.5 mm, 68 parts, among them P1 SOIL, P101 CONN_DIGITAL, P102 CONN_ANALOG, P103 CONN_SERIAL, P104 CONN_I2C, P105 SOLAR, P106 USB_5PIN_SHELL, P109 CONN_PWR, P110 CONN_01X05, P111 UV, P112 TEMP, P113 NEOPIXEL, P114 PIR, Q101 FDN340P, Q201 FDN340P, Q202 FDN340P, Q203 FDN340P, SW101 RESET, SW102 PRGM, SW103 RESET, U101 STM32F042F, U103 ESP-12E, U201 CN3063, U202 MCP6002, U301 BME280, U302 ADXL345

Commit message: Second go at a layout.
Parts:
- removed D102: SS14, FT:DIODE_SMA
- removed MH101, MH102, MH103, MH104: TEST_1P, Connect:1pin
- added REF01: MOUNT, Mounting_Holes:MountingHole_5mm, F.Cu at (63.3, 70.5)
- added REF03: MOUNT, Mounting_Holes:MountingHole_5mm, F.Cu at (45.0, 70.5)
- added REF05: MOUNT, Mounting_Holes:MountingHole_3mm, F.Cu at (32.7, 46.9)
- added REF06: MOUNT, Mounting_Holes:MountingHole_3mm, F.Cu at (75.8, 46.9)
- added REF07: MOUNT, Mounting_Holes:MountingHole_3mm, F.Cu at (75.8, 131.5)
- added REF08: MOUNT, Mounting_Holes:MountingHole_3mm, F.Cu at (32.7, 131.5)
- added SJ101: SJ, FT:SJ_SHORTED, F.Cu at (43.1, 42.8)
- P1: value SOIL -> SOIL MOISTURE
- P103: value CONN_SERIAL -> SERIAL
- P104: value CONN_I2C -> I2C
- P109: value CONN_PWR -> PWR
- P110: value CONN_01X05 -> STM_PGM
- P111: value UV -> UV SENSOR
- P112: value TEMP -> TEMP SENSOR
- P113: value NEOPIXEL -> WS2812
- P114: value PIR -> PIR SENSOR
- REG101: value SPX3819M5-3.3 -> SPX3819M5
- moved P113 205.0 mm to (33.2, 80.9), turned to 270 degrees
- moved D101 198.6 mm to (31.4, 102.0), turned to 270 degrees
- moved F101 196.0 mm to (35.5, 105.7), turned to 90 degrees
- moved R111 185.0 mm to (37.6, 48.6), turned to 0 degrees
- moved R113 181.5 mm to (40.5, 47.7), turned to 90 degrees
- moved R202 181.2 mm to (39.3, 106.6), turned to 90 degrees
- moved R203 178.4 mm to (42.7, 106.6), turned to 90 degrees
- moved U103 175.8 mm to (46.7, 39.8), turned to 0 degrees
- moved LED201 175.8 mm to (39.3, 102.5), turned to 90 degrees
- moved LED202 172.8 mm to (42.8, 102.6), turned to 90 degrees
- moved C203 171.1 mm to (47.5, 93.3), turned to 0 degrees
- moved U301 166.2 mm to (71.4, 105.2)
- moved C301 164.8 mm to (68.7, 105.2), turned to 270 degrees
- moved P114 163.6 mm to (75.3, 66.0)
- moved Q203 162.2 mm to (46.7, 101.1), turned to 90 degrees
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Connections:
- P102 pad 4: (no net) -> /ADC3
- P106 pad 4: (no net) -> Net-(P106-Pad4)
- R101 pad 1: /GPIO0 -> /STM_BOOT
- R111 pad 1: +3V3 -> /ESP_~RESET
- R111 pad 2: /ESP_~RESET -> +3V3
- R112 pad 1: /ESP_~RESET -> /GPIO0
- R112 pad 2: /GPIO16 -> +3V3
- U101 pad 1: /GPIO0 -> /STM_BOOT
- U101 pad 11: /SOIL_1 -> /ADC3
- U101 pad 12: /SOIL_2 -> /SOIL_1
- U101 pad 13: /ESP_~RESET -> /SOIL_2
- U103 pad 10: (no net) -> Net-(U103-Pad10)
- U103 pad 11: (no net) -> Net-(U103-Pad11)
- U103 pad 12: (no net) -> Net-(U103-Pad12)
- U103 pad 13: (no net) -> Net-(U103-Pad13)
- U103 pad 14: (no net) -> Net-(U103-Pad14)
- U103 pad 2: (no net) -> Net-(U103-Pad2)
- U103 pad 9: (no net) -> Net-(U103-Pad9)
- U302 pad 10: (no net) -> Net-(U302-Pad10)
- U302 pad 11: (no net) -> Net-(U302-Pad11)
- U302 pad 3: (no net) -> Net-(U302-Pad3)
- U302 pad 9: (no net) -> Net-(U302-Pad9)
Routing:
- net GND: track 154.1 -> 15.6 mm, vias 62 -> 0
- net /VCC_SENS: track 234.0 -> 118.3 mm
- net /GPIO0: track 136.4 -> 42.8 mm, vias 7 -> 0
- net /ESP_~RESET: track 114.6 -> 24.4 mm, vias 2 -> 0
- net /GPIO2: track 46.9 -> 88.9 mm, vias 4 -> 1
- net /Power/VIN: track 116.6 -> 78.4 mm, vias 2 -> 0
- net /USB_D+: track 79.7 -> 44.2 mm, vias 0 -> 2
- net /USB_D-: track 80.6 -> 45.7 mm
- net /Power/VOUT: track 62.4 -> 28.1 mm
- net /I2C Sensors/I2C_SCL: track 128.5 -> 95.3 mm, vias 5 -> 2
- net /STM_RXD: track 36.5 -> 67.3 mm, vias 2 -> 0
- net /GPIO15: track 82.1 -> 53.0 mm, vias 3 -> 0
- net /I2C Sensors/I2C_SDA: track 125.8 -> 99.6 mm, vias 5 -> 0
- net /STM_TXD: track 39.3 -> 65.4 mm, vias 2 -> 1
- net +3V3: track 225.6 -> 201.3 mm, vias 10 -> 1
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Other:
- board size 97 x 77.5 mm -> 49.6 x 97.6 mm
- net class Default: clearance 0.15 -> 0.2; trace_width 0.15 -> 0.25; via_drill 0.3 -> 0.4
- net class Power removed
- net class USB removed
- rule trace_clearance: 0.15 -> 0.2
- rule trace_min: 0.15 -> 0.2
- board text added: "+3v3"
- board text added: "ESPlant - Version 1.0 https://github.com/mage0r/ESPlant Designed by: John Spencer and Angus Gratton Open Hardware MiniConf, LinuxConf, Geelong, 2016 Made at hackmelbourne.org"
- board text added: "I2C"
- board text added: "PWR"
- board text added: "RST"
- board text added: "RXD"
- board text added: "SCL/4"
- board text added: "SDA/5"
- board text added: "SERIAL"
- board text added: "SOIL_1"
- board text added: "SOIL_2"
- board text added: "SOLAR"
- board text added: "STM_PGM"
- board text added: "TXD"
- board text added: "VCC"
- board text added: "WS2812"
- board text removed: "(GPIO0)"
- board text removed: "+3.3V"
- board text removed: "+VSen"
- board text removed: "/4"
- board text removed: "/5"
- board text removed: "ADC4"
- board text removed: "ADC5"
- board text removed: "Designed for LCA2016 Open Hardware MiniConf by Angus Gratton & John Spencer http://github.com/mage0r/ESPlant TAPR Open Hardware License"
- board text removed: "ESP FLASH"
- board text removed: "ESP RESET"
- board text removed: "ESPlant"
- board text removed: "MAX 7V/1A"
- board text removed: "RX (GPIO3)"
- board text removed: "SOLAR PANEL"
- board text removed: "STM DEBUG"
- board text removed: "STM RESET"
- board text removed: "TX (GPIO1)"
- board text removed: "V1.0B"
- board text removed: "WS2812B LEDS"
- board text removed: "~RST"

Commit message: Ok, all updated I hope
Parts:
- removed R203: 330R, FT:0805
- removed SJ101: SJ, FT:SJ_SHORTED
- added C204: 10uF 16V, FT:1210_CAP, F.Cu at (31.3, 106.1)
- added D102: SS14, FT:DIODE_SMA, F.Cu at (38.6, 130.5)
- added R114: 10K, FT:0603, F.Cu at (63.2, 57.3)
- added R205: 7.15K 1%, FT:0603, F.Cu at (39.4, 89.8)
- added SW104: SS12D00, Plant:SS12D00, F.Cu at (60.2, 100.7)
- added TH201: 10K NTC, FT:0603, F.Cu at (43.7, 90.7)
- C101: value 100nF -> 100nF 6.3V; footprint FT:0805 -> FT:0603_CAP
- C102, C104, C107, C202, C301, C302: footprint FT:0805 -> FT:0603_CAP
- C106: value 220uF 16V -> 100uF 16V X5R
- P1: value SOIL MOISTURE -> SOIL
- P103: value SERIAL -> CONN_SERIAL
- P104: value I2C -> CONN_I2C
- P109: value PWR -> CONN_PWR
- P110: value STM_PGM -> CONN_01X05
- P111: value UV SENSOR -> UV
- P112: value TEMP SENSOR -> TEMP
- P113: value WS2812 -> NEOPIXEL
- P114: value PIR SENSOR -> PIR
- R101: value 10K DNP -> 1K; footprint FT:0805 -> FT:0603
- R102, R103: value 100K -> 100K 1%; footprint FT:0805 -> FT:0603
- R104, R105, R106, R109, R110, R113, R201, R301, R302: footprint FT:0805 -> FT:0603
- R107: value 56K 1% -> 121K 1%; footprint FT:0805 -> FT:0603
- R108: value 47K 1% -> 100K 1%; footprint FT:0805 -> FT:0603
- R112: value 10K -> 1K; footprint FT:0805 -> FT:0603
- R202: value 330R -> 1K; footprint FT:0805 -> FT:0603
- R204: value 8.2K -> 7.15K 1%; footprint FT:0805 -> FT:0603
- REG101: value SPX3819M5 -> SPX3819M5-3.3
- U103: footprint ESP:ESP-12E -> Plant:ESP-12E-no-overhang
- moved R112 30.7 mm to (40.4, 50.0), turned to 0 degrees
- moved P103 30.3 mm to (70.4, 46.2)
- moved R111 5.66 mm to (40.2, 43.6), turned to 90 degrees
- moved C302 4.42 mm to (66.2, 102.5), turned to 180 degrees
- moved R202 3.47 mm to (42.7, 106.4)
- moved R301 2.70 mm to (66.1, 45.8)
- moved R109 2.63 mm to (67.0, 57.3), turned to 0 degrees
- moved R302 2.13 mm to (66.1, 43.7)
- moved D101 1.96 mm to (31.3, 100.1)
- moved P109 1.38 mm to (31.9, 89.6)
- moved R106 1.38 mm to (36.9, 89.7)
- moved R104 1.21 mm to (34.5, 89.7)
- moved R113 0.78 mm to (40.5, 46.9), turned to 0 degrees
- moved C203 0.48 mm to (47.9, 93.0)
- moved R204 0.31 mm to (42.0, 90.7), turned to 90 degrees
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Connections:
- LED202 pad A: Net-(LED202-PadA) -> Net-(LED201-PadA)
- P101 pad 3: /I2C Sensors/I2C_SCL -> /I2C Sensors/I2C_SDA
- P101 pad 4: /I2C Sensors/I2C_SDA -> /I2C Sensors/I2C_SCL
- P102 pad 4: /ADC3 -> /SOIL_1
- P102 pad 5: /SOIL_1 -> /SOIL_2
- P102 pad 6: /SOIL_2 -> GND
- Q101 pad D: +3V3 -> /VCC_SENS
- Q101 pad S: /VCC_SENS -> +3V3
- R101 pad 1: /STM_BOOT -> /GPIO0_BOOT
- R101 pad 2: GND -> /GPIO0
- R105 pad 1: /GPIO2 -> /GPIO13
- R111 pad 1: /ESP_~RESET -> +3V3
- R111 pad 2: +3V3 -> /ESP_~RESET
- R112 pad 1: /GPIO0 -> /ESP_~RESET
- R112 pad 2: +3V3 -> /GPIO16
- REG101 pad 1: /Power/VOUT -> /VSWITCHED
- REG101 pad 3: /Power/VOUT -> /VSWITCHED
- SW102 pad 2: /GPIO0 -> /GPIO0_BOOT
- U101 pad 1: /STM_BOOT -> /GPIO0_BOOT
- U101 pad 11: /ADC3 -> /SOIL_1
- U101 pad 12: /SOIL_1 -> /SOIL_2
- U101 pad 13: /SOIL_2 -> /ESP_~RESET
- U103 pad 19: /I2C Sensors/I2C_SCL -> /I2C Sensors/I2C_SDA
- U103 pad 20: /I2C Sensors/I2C_SDA -> /I2C Sensors/I2C_SCL
- U201 pad 1: GND -> Net-(R205-Pad2)
- U301 pad 5: GND -> +3V3
- U302 pad 12: +3V3 -> GND
Routing:
- net /GPIO2: track 88.9 -> 12.6 mm, vias 1 -> 0
- net /ESP_~RESET: track 24.4 -> 76.9 mm, vias 0 -> 1
- net /GPIO0_BOOT: track 0.00 -> 46.1 mm
- net /GPIO13: track 47.4 -> 84.0 mm, vias 0 -> 1
- net +3V3: track 201.3 -> 229.7 mm, vias 1 -> 2
- net /STM_RXD: track 67.3 -> 84.6 mm, vias 0 -> 1
- net /USB_D+: track 44.2 -> 60.4 mm
- net GND: track 15.6 -> 0.00 mm
- net /GPIO14: track 64.5 -> 51.4 mm
- net /ADC3: track 12.0 -> 0.00 mm
- net /VSWITCHED: track 0.00 -> 11.6 mm, vias 0 -> 1
- net /I2C Sensors/I2C_SCL: track 95.3 -> 85.2 mm, vias 2 -> 0
- net /ADC0: track 38.1 -> 47.5 mm, vias 0 -> 1
- net Net-(R205-Pad2): track 0.00 -> 7.96 mm
- net /Power/SOLAR_IN: track 12.5 -> 20.1 mm
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