File: Circuit/ESPlant.kicad_pcb (KiCad board)
At the start: 2 copper layers, 97 x 77.5 mm, 75 parts, among them P1 SOIL, P101 CONN_DIGITAL, P102 CONN_ANALOG, P103 CONN_SERIAL, P104 CONN_I2C, P105 SOLAR, P106 USB_5PIN_SHELL, P109 CONN_PWR, P110 CONN_01X05, P111 UV, P112 TEMP, P113 NEOPIXEL, P114 PIR, Q101 FDN340P, Q201 FDN340P, Q202 FDN340P, Q203 FDN340P, SW101 RESET, SW102 PRGM, SW103 RESET, SW104 SS12D00, U101 STM32F042F, U103 ESP-12E, U201 CN3063, U202 MCP6002, U301 BME280, U302 ADXL345

Commit message: Fix stray n/c trace, ground CN3063 pad, bump to V1.2
Connections:
- U201 pad PAD: (no net) -> GND
Routing:
- net GND: track 159.3 -> 187.4 mm, vias 66 -> 73
- net (no net): track 4.33 -> 0.00 mm, vias 3 -> 0
Other:
- board text added: "V1.2"
- board text removed: "V1.1"

Commit message: Fix silkscreen & slot width issues noted by @hackvana, bump version V1.3
Other:
- outline, holes or cut-outs redrawn
- board text added: "V1.3"
- board text removed: "V1.2"
Changed lines of the file:
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@@
     (links 189)
     (no_connects 0)
-    (area 141.924999 60.424999 239.075001 138.075001)
+    (area 126.97 50.8 241.300001 138.419)
     (thickness 1.6)
     (drawings 127)
@@
     (add_net /USB_D-)
   )
+  (module Plant:SS12D00 (layer F.Cu)
+    (at 225.8 70.3 90)
+    (fp_text reference SW104 (at 0 -2.6 90) (layer F.SilkS)
+      (effects (font (size 0.8 0.8) (thickness 0.15)))
+    )
+    (fp_text value SS12D00 (at 0 -1.5 90) (layer F.Fab) hide
+      (effects (font (size 1 1) (thickness 0.15)))
+    )
+    (fp_line (start -4.25 1.75) (end -4.25 -1.75) (layer F.SilkS) (width 0.2))
+    (fp_line (start 4.25 1.75) (end -4.25 1.75) (layer F.SilkS) (width 0.2))
+    (fp_line (start 4.25 -1.75) (end 4.25 1.75) (layer F.SilkS) (width 0.2))
+    (fp_line (start -4.25 -1.75) (end 4.25 -1.75) (layer F.SilkS) (width 0.2))
+    (pad 2 thru_hole circle (at 0 0 90) (size 1.6 1.6) (drill 1) (layers *.Cu *.Mask F.SilkS)
+      (net 44 /VSWITCHED))
+    (pad 1 thru_hole circle (at -2.5 0 90) (size 1.6 1.6) (drill 1) (layers *.Cu *.Mask F.SilkS)
+      (net 7 /Power/VOUT))
+    (pad 3 thru_hole circle (at 2.5 0 90) (size 1.6 1.6) (drill 1) (layers *.Cu *.Mask F.SilkS))
+  )
   (module Plant:lca2016_logo (layer B.Cu)
     (at 186.8 82.5 180)
@@
     (descr "<b>Small Outline Package 8</b><br>")
     (fp_text reference U202 (at -3.235 -0.19842 90) (layer F.SilkS)
-      (effects (font (size 0.8 0.8) (thickness 0.125)))
+      (effects (font (size 0.7 0.7) (thickness 0.15)))
     )
     (fp_text value MCP6002 (at 3.35 -0.1 90) (layer F.SilkS) hide
@@
   (module FT:SCREWTERMINAL-3.5MM-3 (layer F.Cu)
     (at 145.5 105.6023 270)
-    (fp_text reference P1 (at -0.2 -1.85 270) (layer F.SilkS)
+    (fp_text reference P1 (at -0.2 -1.85 270) (layer F.SilkS) hide
       (effects (font (size 0.4064 0.4064) (thickness 0.03048)))
     )
@@
   (module FT:SCREWTERMINAL-3.5MM-3 (layer F.Cu)
     (at 235.5 83.6 90)
-    (fp_text reference P112 (at -0.2 -1.85 90) (layer F.SilkS)
+    (fp_text reference P112 (at -0.2 -1.85 90) (layer F.SilkS) hide
       (effects (font (size 0.4064 0.4064) (thickness 0.03048)))
     )
@@
   (module FT:SCREWTERMINAL-3.5MM-2 (layer F.Cu)
     (at 145.5 75.60242 270)
-    (fp_text reference P105 (at 1.6 -1.9 270) (layer F.SilkS)
+    (fp_text reference P105 (at 1.6 -1.9 270) (layer F.SilkS) hide
       (effects (font (size 0.7 0.7) (thickness 0.15)))
     )
@@
   (module FT:SCREWTERMINAL-3.5MM-3 (layer F.Cu)
     (at 235.5 114.0977 90)
-    (fp_text reference P113 (at -0.2 -1.85 90) (layer F.SilkS)
+    (fp_text reference P113 (at -0.2 -1.85 90) (layer F.SilkS) hide
       (effects (font (size 0.4064 0.4064) (thickness 0.03048)))
     )
@@
     (at 153.0988 85.7606 180)
     (descr "<b>OMRON SWITCH</b>")
-    (fp_text reference SW101 (at -0.05 0.0806 180) (layer F.SilkS)
+    (fp_text reference SW101 (at -0.05 3.8606 180) (layer F.SilkS)
       (effects (font (size 0.7 0.7) (thickness 0.15)))
     )
@@
     (at 153.0988 93.6606 180)
     (descr "<b>OMRON SWITCH</b>")
-    (fp_text reference SW102 (at 0.1112 0.0594 180) (layer F.SilkS)
+    (fp_text reference SW102 (at -0.0012 3.8606 180) (layer F.SilkS)
       (effects (font (size 0.7 0.7) (thickness 0.15)))
     )
@@
   (module FT:SCREWTERMINAL-3.5MM-3 (layer F.Cu)
     (at 235.6 98.8977 90)
-    (fp_text reference P114 (at -0.2 -1.85 90) (layer F.SilkS)
+    (fp_text reference P114 (at -0.2 -1.85 90) (layer F.SilkS) hide
       (effects (font (size 0.4064 0.4064) (thickness 0.03048)))
     )
@@
     (pad "" np_thru_hole circle (at -19 -8.2 180) (size 1.8 1.8) (drill 1.8) (layers *.Cu *.Mask F.SilkS))
   )
-  (module Plant:SS12D00 (layer F.Cu)
-    (at 225.8 70.3 90)
-    (fp_text reference SW104 (at 0 -2.6 90) (layer F.SilkS)
-      (effects (font (size 0.8 0.8) (thickness 0.12)))
-    )
-    (fp_text value SS12D00 (at 0 -1.5 90) (layer F.Fab) hide
-      (effects (font (size 1 1) (thickness 0.15)))
-    )
-    (fp_line (start -4.25 1.75) (end -4.25 -1.75) (layer F.SilkS) (width 0.1))
-    (fp_line (start 4.25 1.75) (end -4.25 1.75) (layer F.SilkS) (width 0.1))
-    (fp_line (start 4.25 -1.75) (end 4.25 1.75) (layer F.SilkS) (width 0.1))
-    (fp_line (start -4.25 -1.75) (end 4.25 -1.75) (layer F.SilkS) (width 0.1))
-    (pad 2 thru_hole circle (at 0 0 90) (size 1.6 1.6) (drill 1) (layers *.Cu *.Mask F.SilkS)
-      (net 44 /VSWITCHED))
-    (pad 1 thru_hole circle (at -2.5 0 90) (size 1.6 1.6) (drill 1) (layers *.Cu *.Mask F.SilkS)
-      (net 7 /Power/VOUT))
-    (pad 3 thru_hole circle (at 2.5 0 90) (size 1.6 1.6) (drill 1) (layers *.Cu *.Mask F.SilkS))
-  )
   (module FT:0603_CAP (layer F.Cu)
     (at 217.20084 99.1 180)
@@
     (effects (font (size 1.1 1.1) (thickness 0.2)) (justify left))
   )
-  (gr_line (start 231.3 123.5) (end 237.5 123.5) (layer Edge.Cuts) (width 0.3))
-  (gr_line (start 229 125.8) (end 229 127.2) (layer Edge.Cuts) (width 0.3))
-  (gr_line (start 231.3 123.5) (end 229 125.8) (layer Edge.Cuts) (width 0.3))
+  (gr_line (start 231.3 123.5) (end 238 123.5) (layer Edge.Cuts) (width 0.6))
+  (gr_line (start 229 125.8) (end 229 126.9) (layer Edge.Cuts) (width 0.6))
+  (gr_line (start 231.3 123.5) (end 229 125.8) (layer Edge.Cuts) (width 0.6))
   (gr_text ON (at 228.3 71.9) (layer F.SilkS)
     (effects (font (size 2 2) (thickness 0.4)) (justify left))
@@
     (effects (font (size 1.5 1.5) (thickness 0.25)) (justify right))
   )
-  (gr_text V1.2 (at 171.1 74.5) (layer F.SilkS)
+  (gr_text V1.3 (at 171.1 74.5) (layer F.SilkS)
     (effects (font (size 1 1) (thickness 0.15)) (justify left))
   )
@@
   (gr_arc (start 236.5 63) (end 236.5 60.5) (angle 90) (layer Edge.Cuts) (width 0.15))
   (gr_arc (start 236.5 135.5) (end 239 135.5) (angle 90) (layer Edge.Cuts) (width 0.15))
-  (gr_line (start 229 130) (end 229 129.1) (layer Edge.Cuts) (width 0.3))
-  (gr_line (start 237.5 130) (end 229 130) (layer Edge.Cuts) (width 0.3))
+  (gr_line (start 229 130) (end 229 129.3) (layer Edge.Cuts) (width 0.6))
+  (gr_line (start 238 130) (end 229 130) (layer Edge.Cuts) (width 0.6))
   (gr_text WS2812B (at 237.65 106.6) (layer F.SilkS)
     (effects (font (size 1.5 1.5) (thickness 0.25)) (justify right))

Commit message: Fix labelling of 'WS2812B' screw terminal as GPIO15, is actually GPIO13
Other:
- board text added: "V1.4"
- board text removed: "V1.3"
Changed lines of the file:
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@@
     (effects (font (size 1.1 1.1) (thickness 0.2)) (justify right mirror))
   )
-  (gr_text GPIO15 (at 225.09512 114.20676) (layer B.SilkS)
+  (gr_text GPIO13 (at 225.09512 114.20676) (layer B.SilkS)
     (effects (font (size 1.1 1.1) (thickness 0.2)) (justify right mirror))
   )
@@
     (effects (font (size 1.5 1.5) (thickness 0.25)) (justify right))
   )
-  (gr_text V1.3 (at 171.1 74.5) (layer F.SilkS)
+  (gr_text V1.4 (at 171.1 74.5) (layer F.SilkS)
     (effects (font (size 1 1) (thickness 0.15)) (justify left))
   )
@@
     (effects (font (size 1.1 1.1) (thickness 0.2)) (justify right))
   )
-  (gr_text GPIO15 (at 231 114.2) (layer F.SilkS)
+  (gr_text "GPIO13\n" (at 231 114.2) (layer F.SilkS)
     (effects (font (size 1.1 1.1) (thickness 0.2)) (justify right))
   )

Commit message: Add power selection resistors R203, R206 as "tie breakers" for VBAT=VIN
Closes #4

Bump version V1.5
Parts:
- added R203: 100K, FT:0603, F.Cu at (209.2, 96.1)
- added R206: 100K, FT:0603, F.Cu at (206.5, 96.1)
- C101, C102, C107: value 100nF 6.3V -> 100nF
- C202: value 100nF -> 100nF 16V
- C301, C302: value 1uF 6.3V -> 1uF
Routing:
- net GND: track 187.4 -> 204.5 mm, vias 73 -> 78
- net /Power/GBAT: track 19.5 -> 26.5 mm, vias 2 -> 0
- net /Power/VOUT: track 80.9 -> 83.0 mm
- net /Power/GIN: track 17.8 -> 19.8 mm
- net /Power/VIN: track 109.3 -> 108.2 mm, vias 2 -> 0
Other:
- rule trace_min: 0.15 -> 0
- board text added: "V1.5"
- board text removed: "V1.4"
